File: hardware/hardware-board/openchess-board.kicad_sch (KiCad schematic)
At the start: 248 parts, among them J1 Conn_02x13, U1 A3144, U10 A3144, U11 A3144, U12 A3144, U13 A3144, U14 A3144, U15 A3144, U16 A3144, U17 A3144, U18 A3144, U19 A3144, U2 A3144, U20 A3144, U21 A3144, U22 A3144, U23 A3144, U24 A3144, U25 A3144, U26 A3144, U27 A3144, U28 A3144, U29 A3144, U3 A3144, U30 A3144, U31 A3144, U32 A3144, U33 A3144, U34 A3144, U35 A3144, U36 A3144, U37 A3144, U38 A3144, U39 A3144, U4 A3144, U40 A3144, U41 A3144, U42 A3144, U43 A3144, U44 A3144, U45 A3144, U46 A3144, U47 A3144, U48 A3144, U49 A3144, U5 A3144, U50 A3144, U51 A3144, U52 A3144, U53 A3144, U54 A3144, U55 A3144, U56 A3144, U57 A3144, U58 A3144, U59 A3144, U6 A3144, U60 A3144, U61 A3144, U62 A3144, U63 A3144, U64 A3144, U7 A3144, U8 A3144, U9 A3144

Commit message: Add new mechanical and power symbols for schematic integration
- Introduced new symbols: TestPoint, Fiducial, MountingHole, +3V3, and GND.
- Each symbol includes properties for reference, value, footprint, datasheet, description, keywords, and filters.
- Implemented a Python script to merge test/mech snippets into the main schematic, ensuring backup and validation of parens.
- The script adds missing symbol definitions and integrates component instances, labels, wires, and power ports.
Parts:
- J1: footprint Connector_PinHeader_2.54mm:PinHeader_2x13_P2.54mm_Vertical -> (none)

Commit message: Add PCB layout and schematic guides for OpenChess controller
- Introduced `controller-PCB_LAYOUT_GUIDE.planning.md` detailing PCB layout constraints, component placement zones, net classes, routing priorities, and mechanical verification for the OpenChess controller.
- Added `controller-SCHEMATIC_GUIDE.planning.md` providing a comprehensive schematic specification, including reference designators, net lists, component details, and validation rules for the OpenChess controller PCB.
Parts:
- removed C91: 470uF, Capacitor_THT:CP_Radial_D10.0mm_P5.00mm, symbol Device:C_Polarized
- U1, U10, U11, U12, U13, U14, U15, U16, U17, U18, U19, U2, U20, U21, U22, U23, U24, U25, U26, U27, U28, U29, U3, U30, U31, U32, U33, U34, U35, U36, U37, U38, U39, U4, U40, U41, U42, U43, U44, U45, U46, U47, U48, U49, U5, U50, U51, U52, U53, U54, U55, U56, U57, U58, U59, U6, U60, U61, U62, U63, U64, U7, U8, U9: value A3144 -> DRV5032FC; footprint Package_TO_SOT_THT:TO-92_Inline -> Package_TO_SOT_SMD:SOT-23

Commit message: Add initial files for openchess board project
- Created Gerber job file for openchess board with specifications and material stackup.
- Added backup of the KiCad PCB file before modifications.
- Introduced STEP files for the 3x3 chess board and the main chess controller.
- Initialized notes file for project documentation.
Parts:
- J1: footprint (none) -> Connector_PinHeader_2.54mm:PinHeader_2x13_P2.54mm_Vertical
Changed lines of the file:
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@@
 			)
 		)
-		(property "Footprint" ""
+		(property "Footprint" "Connector_PinHeader_2.54mm:PinHeader_2x13_P2.54mm_Vertical"
 			(at 377.19 353.06 0)
 			(hide yes)

Commit message: Add scripts to merge and tile PDF layers for KiCad projects
- Implemented `merge_pdf_layers.py` to overlay multiple single-page PDFs into one page, allowing for easy printing of layered designs.
- Created `tile_pdf_to_a4.py` to split large PDFs into A4-sized tiles with configurable overlap, facilitating printing on standard home printers.
- Both scripts require the `pypdf` library for PDF manipulation.
Parts:
- removed FID1, FID2, FID3: Fiducial, Fiducial:Fiducial_1mm_Mask2mm, symbol Mechanical:Fiducial
- removed MH1, MH2, MH3, MH4: M3, MountingHole:MountingHole_3.2mm_M3, symbol Mechanical:MountingHole
- removed TP1, TP2, TP3, TP4: TestPoint, TestPoint:TestPoint_Pad_D1.5mm, symbol Connector:TestPoint
