File: hardware/hardware-controller-v2/openchess-controller.kicad_sch (KiCad schematic)
At the start: 71 parts, among them J1 Conn_02x13, J4 TYPE-C-31-M-12, J5 B2B-XH-A, J6 J_OLED XH-4, J7 J_BTN_UP XH-2, J8 J_BTN_DOWN XH-2, J9 J_BTN_OK XH-2, Q1 S8050 J3Y, Q2 S8050 J3Y, SW1 MSK12C02, U10 TPS61022RWUR, U11 AMS1117-3.3, U2 ESP32-WROOM-E, U3 74AHCT125, U6 TBD62783A, U7 CH340C, U8 USBLC6-2SC6, U9 BQ24074RGTR

Commit message: fix(hw): v2 review fixes — R1-R8 LCSC to 0805 part C17414, R11 C23140, BTN_OK rename
- R1-R8 (10k, 0805 footprints) LCSC changed C25804 -> C17414, the 0805-body
  10k from the v1 production BOM (physically validated); C25804 (0603) now
  only on R20/R23/R24/R30/R36/R37
- R11 (33Ω 0603): add LCSC C23140 (v1-proven part)
- docs/gpio-map.md v2 section: rename two leftover BTN_SELECT occurrences
  to BTN_OK (design-rules prose + v2 pin table, J9 noted); v1 untouched
- ERC 0 violations; check_task6 45/45; check_task7 89/89

Co-Authored-By: Claude Fable 5 <noreply@anthropic.com>
Parts:
- R1, R2, R3, R4, R5, R6, R7, R8: LCSC C25804 -> C17414
- R11: LCSC (none) -> C23140
Changed lines of the file:
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@@
 			)
 		)
+		(property "LCSC" "C23140"
+			(at 177.8 200.66 0)
+			(hide yes)
+			(show_name no)
+			(do_not_autoplace no)
+			(effects
+				(font
+					(size 1.27 1.27)
+				)
+			)
+		)
 		(property "Datasheet" ""
 			(at 177.8 200.66 0)
@@
 			)
 		)
-		(property "LCSC" "C25804"
+		(property "LCSC" "C17414"
 			(at 233.68 91.44 0)
 			(hide yes)
@@
 			)
 		)
-		(property "LCSC" "C25804"
+		(property "LCSC" "C17414"
 			(at 212.09 91.44 0)
 			(hide yes)
@@
 			)
 		)
-		(property "LCSC" "C25804"
+		(property "LCSC" "C17414"
 			(at 186.69 91.44 0)
 			(hide yes)
@@
 			)
 		)
-		(property "LCSC" "C25804"
+		(property "LCSC" "C17414"
 			(at 163.83 91.44 0)
 			(hide yes)
@@
 			)
 		)
-		(property "LCSC" "C25804"
+		(property "LCSC" "C17414"
 			(at 198.12 91.44 0)
 			(hide yes)
@@
 			)
 		)
-		(property "LCSC" "C25804"
+		(property "LCSC" "C17414"
 			(at 175.26 91.44 0)
 			(hide yes)
@@
 			)
 		)
-		(property "LCSC" "C25804"
+		(property "LCSC" "C17414"
 			(at 152.4 91.44 0)
 			(hide yes)
@@
 			)
 		)
-		(property "LCSC" "C25804"
+		(property "LCSC" "C17414"
 			(at 223.52 91.44 0)
 			(hide yes)
