File: hardware/hardware-controller-v2/openchess-controller.kicad_pcb (KiCad board)
At the start: 2 copper layers, 58 x 71 mm, 28 parts, among them J1 Conn_02x13, J3 J_PANEL XH-10, M1 Lipo Rider Plus, U2 ESP32-DevKitC, U3 74AHCT125, U6 TBD62783A

Commit message: docs: refresh repo for public
Parts:
- removed D2: SS14 (or BAT60A), Diode_SMD:D_SMA
- removed FID1, FID2, FID3: Fiducial, Fiducial:Fiducial_1mm_Mask2mm
- removed J3: J_PANEL XH-10, Connector_PinHeader_2.54mm:PinHeader_1x10_P2.54mm_Vertical
- removed M1: Lipo Rider Plus, Connector_PinSocket_2.54mm:PinSocket_1x08_P2.54mm_Vertical
- added C13: 100nF, Capacitor_SMD:C_0603_1608Metric, F.Cu at (197.1, 45.5)
- added C14: 10µF, Capacitor_SMD:C_0805_2012Metric, F.Cu at (196.9, 43.5)
- added C15: 1µF, Capacitor_SMD:C_0603_1608Metric, F.Cu at (197.2, 47.5)
- added C16: 100nF, Capacitor_SMD:C_0603_1608Metric, F.Cu at (133.4, 100.0)
- added C17: 10µF, Capacitor_SMD:C_0805_2012Metric, F.Cu at (152.5, 74.1)
- added C18: 10µF, Capacitor_SMD:C_0805_2012Metric, F.Cu at (156.9, 68.1)
- added C19: 100nF, Capacitor_SMD:C_0603_1608Metric, F.Cu at (133.4, 92.6)
- added C20: 10µF, Capacitor_SMD:C_0805_2012Metric, F.Cu at (163.8, 20.6)
- added C21: 10µF, Capacitor_SMD:C_0805_2012Metric, F.Cu at (163.8, 23.6)
- added C22: 10µF, Capacitor_SMD:C_0805_2012Metric, F.Cu at (93.3, 47.8)
- added C23: 100µF, Capacitor_SMD:CP_Elec_6.3x5.4, F.Cu at (99.2, 63.1)
- added C24: 22µF, Capacitor_SMD:C_0805_2012Metric, F.Cu at (94.5, 54.8)
- added C25: 22µF, Capacitor_SMD:C_0805_2012Metric, F.Cu at (92.1, 54.8)
- added D4: D, LED_SMD:LED_0603_1608Metric, F.Cu at (164.0, 35.6)
- added D5: D, LED_SMD:LED_0603_1608Metric, F.Cu at (157.2, 88.8)
- added J4: TYPE-C-31-M-12, Connector_USB:USB_C_Receptacle_HRO_TYPE-C-31-M-12, F.Cu at (124.2, 96.5)
- added J5: B2B-XH-A, Connector_JST:JST_XH_B2B-XH-A_1x02_P2.50mm_Vertical, F.Cu at (140.6, 46.5)
- added J6: J_OLED XH-4, Connector_JST:JST_XH_B4B-XH-A_1x04_P2.50mm_Vertical, F.Cu at (135.2, 126.8)
- added J7: J_BTN_UP XH-2, Connector_JST:JST_XH_B2B-XH-A_1x02_P2.50mm_Vertical, F.Cu at (125.5, 118.5)
- added J8: J_BTN_DOWN XH-2, Connector_JST:JST_XH_B2B-XH-A_1x02_P2.50mm_Vertical, F.Cu at (135.2, 118.5)
- added J9: J_BTN_OK XH-2, Connector_JST:JST_XH_B2B-XH-A_1x02_P2.50mm_Vertical, F.Cu at (125.5, 126.8)
- added L1: 1µH, Inductor_SMD:L_APV_APH0420, F.Cu at (108.5, 57.3)
- added Q1: S8050 J3Y, Package_TO_SOT_SMD:SOT-23, F.Cu at (146.9, 94.0)
- added Q2: S8050 J3Y, Package_TO_SOT_SMD:SOT-23, F.Cu at (146.9, 98.4)
- added R20: 10k, Resistor_SMD:R_0603_1608Metric, F.Cu at (197.2, 49.1)
- added R21: 5.1k, Resistor_SMD:R_0603_1608Metric, F.Cu at (131.0, 92.6)
- added R22: 5.1k, Resistor_SMD:R_0603_1608Metric, F.Cu at (131.0, 100.0)
- added R23: 10k, Resistor_SMD:R_0603_1608Metric, F.Cu at (143.7, 94.0)
- added R24: 10k, Resistor_SMD:R_0603_1608Metric, F.Cu at (143.7, 98.4)
- added R25: 1k, Resistor_SMD:R_0603_1608Metric, F.Cu at (151.1, 24.9)
- added R26: 100k, Resistor_SMD:R_0603_1608Metric, F.Cu at (87.0, 52.1)
- added R27: 1k, Resistor_SMD:R_0603_1608Metric, F.Cu at (144.3, 80.4)
- added R28: 1.1K, Resistor_SMD:R_0603_1608Metric, F.Cu at (155.1, 17.3)
- added R29: 910Ω, Resistor_SMD:R_0603_1608Metric, F.Cu at (155.1, 19.8)
- added R30: 10k, Resistor_SMD:R_0603_1608Metric, F.Cu at (155.1, 22.3)
- added R31: 750k, Resistor_SMD:R_0603_1608Metric, F.Cu at (96.8, 50.1)
- added R32: 100k, Resistor_SMD:R_0603_1608Metric, F.Cu at (96.8, 51.9)
- added SW1: MSK12C02, Button_Switch_SMD:SW_SPDT_Shouhan_MSK12C02, F.Cu at (85.6, 48.4)
- added SW_BOOT1: SW_Push, Button_Switch_SMD:SW_Push_1P1T_XKB_TS-1187A, F.Cu at (125.7, 104.8)
- added SW_EN1: SW_Push, Button_Switch_SMD:SW_Push_1P1T_XKB_TS-1187A, F.Cu at (125.7, 88.3)
- added U10: TPS61022RWUR, Package_DFN_QFN:Texas_RWU0007A_VQFN-7_2x2mm_P0.5mm, F.Cu at (93.2, 50.9)
- added U11: AMS1117-3.3, Package_TO_SOT_SMD:SOT-223-3_TabPin2, F.Cu at (165.2, 89.8)
- added U7: CH340C, Package_SO:SOIC-16_3.9x9.9mm_P1.27mm, F.Cu at (138.4, 96.3)
- added U8: USBLC6-2SC6, Package_TO_SOT_SMD:SOT-23-6, F.Cu at (132.2, 96.1)
- added U9: BQ24074RGTR, Package_DFN_QFN:VQFN-16-1EP_3x3mm_P0.5mm_EP1.6x1.6mm_ThermalVias, F.Cu at (152.1, 33.8)
- U2: value ESP32-DevKitC -> ESP32-WROOM-E; footprint Espressif:ESP32-DevKitC -> RF_Module:ESP32-WROOM-32E
- U6: footprint Package_DIP:DIP-18_W7.62mm -> Package_SO:SOP-18_7.495x11.515mm_P1.27mm
- moved R11 166.5 mm to (217.3, 79.3), turned to 0 degrees
- moved C5 155.9 mm to (217.5, 76.5), turned to 0 degrees
- moved U3 155.1 mm to (211.1, 80.3)
- moved U2 142.9 mm to (208.8, 47.6)
- moved R36 110.0 mm to (150.2, 127.1)
- moved R37 109.9 mm to (150.2, 129.6)
- moved U6 109.4 mm to (180.3, 107.0), turned to -90 degrees
- moved J1 109.0 mm to (207.0, 120.0), turned to 90 degrees
- moved R8 108.5 mm to (189.2, 113.5), turned to -90 degrees
- moved R6 106.0 mm to (191.7, 113.5), turned to -90 degrees
- moved R2 105.4 mm to (196.8, 113.5), turned to -90 degrees
- moved R4 105.4 mm to (194.3, 113.5), turned to -90 degrees
- moved R7 105.1 mm to (189.2, 109.0), turned to -90 degrees
- moved R1 103.7 mm to (196.8, 109.0), turned to -90 degrees
- moved R3 102.4 mm to (194.3, 109.0), turned to -90 degrees
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Connections:
- R14 pad 1: /BAT -> /VBAT
- R36 pad 2: /BTN_POWER -> /BTN_UP
- R37 pad 2: /BTN_MODE -> /BTN_DOWN
- U2 pad 1: unconnected-(U2-3V3-Pad1) -> GND
- U2 pad 10: /COL_DRV_D -> /COL_DRV_E
- U2 pad 11: /COL_DRV_C -> /COL_DRV_D
- U2 pad 12: /COL_DRV_B -> /COL_DRV_C
- U2 pad 13: unconnected-(U2-MTDI/GPIO12/ADC2_CH5-Pad13) -> /COL_DRV_B
- U2 pad 14: GND -> /COL_DRV_H
- U2 pad 15: /COL_DRV_A -> GND
- U2 pad 16: unconnected-(U2-SD_DATA2/GPIO9-Pad16) -> /COL_DRV_A
- U2 pad 17: unconnected-(U2-SD_DATA3/GPIO10-Pad17) -> (no net)
- U2 pad 18: unconnected-(U2-CMD-Pad18) -> (no net)
- U2 pad 19: Net-(D2-K) -> (no net)
- U2 pad 2: unconnected-(U2-CHIP_PU-Pad2) -> +3.3V
- U2 pad 20: unconnected-(U2-SD_CLK/GPIO6-Pad20) -> (no net)
- U2 pad 21: unconnected-(U2-SD_DATA0/GPIO7-Pad21) -> (no net)
- U2 pad 22: unconnected-(U2-SD_DATA1/GPIO8-Pad22) -> (no net)
- U2 pad 23: /COL_DRV_H -> /S6
- U2 pad 24: /BTN_SELECT -> /BTN_OK
- U2 pad 25: unconnected-(U2-GPIO0/BOOT/ADC2_CH1-Pad25) -> /IO0
- U2 pad 26: /S0 -> /COL_DRV_G
- U2 pad 27: /S1 -> /S0
- U2 pad 28: /S2 -> /S1
- U2 pad 29: /COL_DRV_G -> /S5
- U2 pad 3: /BTN_POWER -> /EN
- U2 pad 30: /S3 -> /S2
- U2 pad 31: /S4 -> /S3
- U2 pad 32: GND -> (no net)
- U2 pad 33: /S5 -> /I2C_SDA
- U2 pad 34: /I2C_SCL -> /U0RXD
- U2 pad 35: /I2C_SDA -> /U0TXD
- U2 pad 36: /S6 -> /I2C_SCL
- U2 pad 37: /S7 -> /S4
- U2 pad 4: /BTN_MODE -> /BTN_UP
- U2 pad 5: /VBAT_MON -> /BTN_DOWN
- U2 pad 6: /PANEL_SPARE -> /VBAT_MON
- U2 pad 7: /LED_DATA -> /S7
- U2 pad 8: /COL_DRV_F -> /LED_DATA
- U2 pad 9: /COL_DRV_E -> /COL_DRV_F
Routing:
- net +5V_LED: track 286.9 -> 2.34 mm
- net +3.3V: track 157.9 -> 0.00 mm
- net /LED_DATA: track 68.3 -> 0.00 mm, vias 2 -> 0
- net /LED_DATA_5V: track 62.7 -> 0.00 mm, vias 1 -> 0
- net /S7: track 57.1 -> 3.02 mm
- net /COL_DRV_F: track 50.5 -> 0.00 mm
- net /COL_DRV_E: track 46.8 -> 0.00 mm
- net /S6: track 58.4 -> 11.7 mm, vias 2 -> 1
- net /BTN_POWER: track 44.1 -> 0.00 mm
- net /BTN_MODE: track 44.1 -> 0.00 mm
- net /COL_DRV_D: track 42.9 -> 0.00 mm
- net /BTN_SELECT: track 40.1 -> 0.00 mm
- net /PANEL_SPARE: track 39.9 -> 0.00 mm
- net /COL_DRV_G: track 39.7 -> 0.00 mm
- net /COL_DRV_C: track 39.3 -> 0.00 mm
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- removed copper zone on B.Cu, net GND
- removed copper zone on F.Cu, net GND
Other:
- board outline removed
- board text removed: "1"
- board text removed: "B_M"
- board text removed: "B_P"
- board text removed: "B_S"
- board text removed: "Github PaoloJN Controller v0.1"
- board text removed: "PN: 06-07-2026"
- board text removed: "R1"
- board text removed: "R8"
- board text removed: "SCL"
- board text removed: "SDA"
